File: pcb/CI-Test.kicad_sch (KiCad schematic)
At the start: 4 parts, among them J1 Conn_01x01, J2 Conn_01x01

Commit message: fix: another test
Other:
- note added: "blabla"
Changed lines of the file:
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@@
 	(generator_version "8.0")
 	(paper "A4")
-    (title_block
-                (title "CI-Test")
-                (date "${DATE}")
-                (rev "${VERSION}")
-                (company "Qetesh")
-            )
+	(title_block
+		(title "CI-Test")
+		(date "${DATE}")
+		(rev "${VERSION}")
+		(company "Qetesh")
+	)
 	(wire
 		(pts
@@
 		)
 	)
+	(text "blabla"
+		(exclude_from_sim no)
+		(at 171.704 82.55 0)
+		(effects
+			(font
+				(size 1.27 1.27)
+			)
+		)
+	)

Commit message: fix: aaand another one
Other:
- note added: "blablabla"
- note removed: "blabla"
Changed lines of the file:
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@@
 		)
 	)
-	(text "blabla"
+	(text "blablabla"
 		(exclude_from_sim no)
 		(at 171.704 82.55 0)

Commit message: fix: testfix
Other:
- note added: "blabla"
- note removed: "blablabla"
Changed lines of the file:
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@@
 		)
 	)
-	(text "blablabla"
+	(text "blabla\n\n"
 		(exclude_from_sim no)
 		(at 171.704 82.55 0)

Commit message: feat: bla
Other:
- note added: "blabla bla"
- note removed: "blabla"
Changed lines of the file:
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@@
 		)
 	)
-	(text "blabla\n\n"
+	(text "blabla\n\nbla"
 		(exclude_from_sim no)
 		(at 171.704 82.55 0)
